Commit message: Repository refactored

File: src/uav_description/urdf/uav.urdf (robot description, URDF)
Before this commit: robot X650_UAV, 20 links, 19 joints
Links:
- link back_arm_ccw_link: geometry collision mesh filename=package://uav_description/meshes/back_arm_ccw_link.STL; visual mesh filename=package://uav_description/meshes/back_arm_ccw_link.STL
- link back_arm_cw_link: geometry collision mesh filename=package://uav_description/meshes/back_arm_cw_link.STL; visual mesh filename=package://uav_description/meshes/back_arm_cw_link.STL
- link back_motor_ccw_link: geometry collision mesh filename=package://uav_description/meshes/back_motor_ccw_link.STL; visual mesh filename=package://uav_description/meshes/back_motor_ccw_link.STL
- link back_motor_cw_link: geometry collision mesh filename=package://uav_description/meshes/back_motor_cw_link.STL; visual mesh filename=package://uav_description/meshes/back_motor_cw_link.STL
- link back_prop_ccw_link: geometry collision mesh filename=package://uav_description/meshes/back_prop_ccw_link.STL; visual mesh filename=package://uav_description/meshes/back_prop_ccw_link.STL
- link back_prop_cw_link: geometry collision mesh filename=package://uav_description/meshes/back_prop_cw_link.STL; visual mesh filename=package://uav_description/meshes/back_prop_cw_link.STL
- link base_link: geometry collision mesh filename=package://uav_description/meshes/base_link.STL; visual mesh filename=package://uav_description/meshes/base_link.STL
- link depth_camera_link: geometry collision mesh filename=package://uav_description/meshes/depth_camera_link.STL; visual mesh filename=package://uav_description/meshes/depth_camera_link.STL
- link front_arm_ccw_link: geometry collision mesh filename=package://uav_description/meshes/front_arm_ccw_link.STL; visual mesh filename=package://uav_description/meshes/front_arm_ccw_link.STL
- link front_arm_cw_link: geometry collision mesh filename=package://uav_description/meshes/front_arm_cw_link.STL; visual mesh filename=package://uav_description/meshes/front_arm_cw_link.STL
- link front_motor_ccw_link: geometry collision mesh filename=package://uav_description/meshes/front_motor_ccw_link.STL; visual mesh filename=package://uav_description/meshes/front_motor_ccw_link.STL
- link front_motor_cw_link: geometry collision mesh filename=package://uav_description/meshes/front_motor_cw_link.STL; visual mesh filename=package://uav_description/meshes/front_motor_cw_link.STL
- link front_prop_ccw_link: geometry collision mesh filename=package://uav_description/meshes/front_prop_ccw_link.STL; visual mesh filename=package://uav_description/meshes/front_prop_ccw_link.STL
- link front_prop_cw_link: geometry collision mesh filename=package://uav_description/meshes/front_prop_cw_link.STL; visual mesh filename=package://uav_description/meshes/front_prop_cw_link.STL
- link gps_module_link: geometry collision mesh filename=package://uav_description/meshes/gps_module_link.STL; visual mesh filename=package://uav_description/meshes/gps_module_link.STL
- link left_landing_gear_link: geometry collision mesh filename=package://uav_description/meshes/left_landing_gear_link.STL; visual mesh filename=package://uav_description/meshes/left_landing_gear_link.STL
- link lidar_link: geometry collision mesh filename=package://uav_description/meshes/lidar_link.STL; visual mesh filename=package://uav_description/meshes/lidar_link.STL
- link pixhawk_jetson_mc_link: geometry collision mesh filename=package://uav_description/meshes/pixhawk_jetson_mc_link.STL; visual mesh filename=package://uav_description/meshes/pixhawk_jetson_mc_link.STL
- link right_landing_gear_link: geometry collision mesh filename=package://uav_description/meshes/right_landing_gear_link.STL; visual mesh filename=package://uav_description/meshes/right_landing_gear_link.STL
- link telemetry_link: geometry collision mesh filename=package://uav_description/meshes/telemetry_link.STL; visual mesh filename=package://uav_description/meshes/telemetry_link.STL
