Commit message: Laser scan and camera issue fixed.

File: src/uav_description/urdf/uav.urdf.xacro (robot description, xacro)
@@ -3,441 +3,688 @@
      Commit Version: 1.6.0-4-g7f85cfe  Build Version: 1.6.7995.38578
      For more information, please see http://wiki.ros.org/sw_urdf_exporter -->
-<robot name="UAV_X650" xmlns:xacro="http://www.ros.org/wiki/xacro">
+<robot name="uav_uav" xmlns:xacro="http://www.ros.org/wiki/xacro">
   <xacro:include filename="$(find uav_description)/urdf/core.xacro"/>
   <xacro:include filename="$(find uav_description)/urdf/uav.gazebo.xacro"/>
-  <link name="x650_0/base_footprint"/>
-  <joint name="x650_0/base_footprint_joint" type="fixed">
-    <origin xyz="0 0 0" rpy="0 0 0" />
-    <parent link="x650_0/base_footprint" />
-    <child link="x650_0/base_link" />
-  </joint>
-  <link name="x650_0/base_link">
-    <inertial>
-      <origin
-        xyz="-0.00372276524577257 -0.00744305903269664 8.57191257253331E-05"
-        rpy="0 0 0" />
-      <mass
-        value="2.79538458384779" />
-      <inertia
-        ixx="0.00251955261705473"
-        ixy="-1.69520154890596E-05"
-        ixz="-9.26102151476342E-05"
-        iyy="0.00725324885475083"
-        iyz="5.60750810648567E-06"
-        izz="0.00570366183964889" />
-    </inertial>
-    <visual>
-      <origin xyz="0 0 0" rpy="0 0 0" />
-      <geometry>
-        <mesh
-          filename="file://$(find uav_description)/meshes/base_link.STL" />
-      </geometry>
-      <material
-        name="">
-        <color
-          rgba="0.752941176470588 0.752941176470588 0.752941176470588 1" />
-      </material>
-    </visual>
-    <collision>
-      <origin
-        xyz="0 0 0"
-        rpy="0 0 0" />
-      <geometry>
-        <mesh
-          filename="file://$(find uav_description)/meshes/base_link.STL" />
-      </geometry>
-    </collision>
-  </link>
-  <link
-    name="x650_0/lidar_link">
-    <inertial>
-      <origin
-        xyz="4.8942772647276E-06 -4.43974432931928E-06 -1.38118108244933E-06"
-        rpy="0 0 0" />
-      <mass
-        value="0.176960287140508" />
-      <inertia
-        ixx="8.43864963091213E-05"
-        ixy="5.21487883463066E-08"
-        ixz="2.33776252508404E-06"
-        iyy="8.04534800729579E-05"
-        iyz="3.09845357754836E-08"
-        izz="0.00011764358096126" />
-    </inertial>
-    <visual>
-      <origin
-        xyz="0 0 0"
-        rpy="0 0 0" />
-      <geometry>
-        <mesh
-          filename="file://$(find uav_description)/meshes/lidar_link.STL" />
-      </geometry>
-      <material
-        name="">
-        <color
-          rgba="1 1 1 0.35" />
-      </material>
-    </visual>
-    <collision>
-      <origin
-        xyz="0 0 0"
-        rpy="0 0 0" />
-      <geometry>
-        <mesh
-          filename="file://$(find uav_description)/meshes/lidar_link.STL" />
-      </geometry>
-    </collision>
-  </link>
-  <joint
-    name="x650_0/lidar_joint"
-    type="fixed">
-    <origin
-      xyz="-0.00044268 -0.00016922 0.12747"
-      rpy="0.0038504 -0.0036204 -0.013619" />
-    <parent
-      link="x650_0/base_link" />
-    <child
-      link="x650_0/lidar_link" />
-    <axis
-      xyz="0 0 0" />
-  </joint>
-  <!-- LiDAR link -->
-  <link name="x650_0/laser_sensor_link">
-    <visual>
-      <geometry>
-        <cylinder radius="0.02" length="0.03"/>
-      </geometry>
-    </visual>
-  </link>
-  <joint name="x650_0/laser_sensor_joint" type="fixed">
-    <parent link="x650_0/base_link"/>
-    <child link="x650_0/laser_sensor_link"/>
-    <origin xyz="0 0 0.15" rpy="0 0 0"/>
-  </joint>
-  <link
-    name="x650_0/gps_module_link">
-    <inertial>
-      <origin
-        xyz="3.55581267098143E-06 3.11348564280278E-06 0.0074610663167827"
-        rpy="0 0 0" />
-      <mass
-        value="0.0240695000069686" />
-      <inertia
-        ixx="3.50312288057669E-06"
-        ixy="-4.71416518047791E-12"
-        ixz="-8.33177101340744E-12"
-        iyy="3.47761888412337E-06"
-        iyz="1.85176336280484E-09"
-        izz="6.33826733013106E-06" />
-    </inertial>
-    <visual>
-      <origin
-        xyz="0 0 0"
-        rpy="0 0 0" />
-      <geometry>
-        <mesh
-          filename="file://$(find uav_description)/meshes/gps_module_link.STL" />
-      </geometry>
-      <material
-        name="">
-        <color
-          rgba="1 1 1 0.35" />
-      </material>
-    </visual>
-    <collision>
-      <origin
-        xyz="0 0 0"
-        rpy="0 0 0" />
-      <geometry>
-        <mesh
-          filename="file://$(find uav_description)/meshes/gps_module_link.STL" />
-      </geometry>
-    </collision>
-  </link>
-  <joint
-    name="x650_0/gps_module_joint"
-    type="fixed">
-    <origin
-      xyz="-0.13598 0.0015189 0.10049"
-      rpy="0.0025723 0.004617 -1.8307" />
-    <parent
-      link="x650_0/base_link" />
-    <child
-      link="x650_0/gps_module_link" />
-    <axis
-      xyz="0 0 0" />
-  </joint>
-  <link
-    name="x650_0/front_prop_ccw_link">
-    <inertial>
-      <origin
-        xyz="1.9285E-05 -0.0005696 0.0086392"
-        rpy="0 0 0" />
-      <mass
-        value="0.023288" />
-      <inertia
-        ixx="7.8138E-07"
-        ixy="-1.9303E-06"
-        ixz="-5.8432E-08"
-        iyy="2.8365E-05"
-        iyz="-3.958E-08"
-        izz="2.9095E-05" />
-    </inertial>
-    <visual>
-      <origin
-        xyz="0 0 0"
-        rpy="0 0 0" />
-      <geometry>
-        <mesh
-          filename="file://$(find uav_description)/meshes/front_prop_ccw_link.STL" />
-      </geometry>
-      <material
-        name="">
-        <color
-          rgba="0.75294 0.75294 0.75294 1" />
-      </material>
-    </visual>
-    <collision>
-      <origin
-        xyz="0 0 0"
-        rpy="0 0 0" />
-      <geometry>
-        <mesh
-          filename="file://$(find uav_description)/meshes/front_prop_ccw_link.STL" />
-      </geometry>
-    </collision>
-  </link>
-  <joint
-    name="x650_0/front_prop_ccw_joint"
-    type="continuous">
-    <origin
-      xyz="0.22481 -0.23326 0.086028"
-      rpy="0 0 0" />
-    <parent
-      link="x650_0/base_link" />
-    <child
-      link="x650_0/front_prop_ccw_link" />
-    <axis
-      xyz="0 0 1" />
-    <limit effort="1e12" velocity="1e12"/>
-    <dynamics damping="0.0" friction="0.0"/>
-  </joint>
-  <link
-    name="x650_0/front_prop_cw_link">
-    <inertial>
-      <origin
-        xyz="1.89889458346304E-06 -0.000131188965704798 0.00588670324654172"
-        rpy="0 0 0" />
-      <mass
-        value="0.0232860557198823" />
-      <inertia
-        ixx="6.48761674575812E-07"
-        ixy="-1.71419194967408E-07"
-        ixz="1.28654962833368E-10"
-        iyy="2.84759689374051E-05"
-        iyz="5.39216374404741E-11"
-        izz="2.90785252715597E-05" />
-    </inertial>
-    <visual>
-      <origin
-        xyz="0 0 0"
-        rpy="0 0 0" />
-      <geometry>
-        <mesh
-          filename="file://$(find uav_description)/meshes/front_prop_cw_link.STL" />
-      </geometry>
-      <material
-        name="">
-        <color
-          rgba="0.752941176470588 0.752941176470588 0.752941176470588 1" />
-      </material>
-    </visual>
-    <collision>
-      <origin
-        xyz="0 0 0"
-        rpy="0 0 0" />
-      <geometry>
-        <mesh
-          filename="file://$(find uav_description)/meshes/front_prop_cw_link.STL" />
-      </geometry>
-    </collision>
-  </link>
-  <joint
-    name="x650_0/front_prop_cw_joint"
-    type="continuous">
-    <origin
-      xyz="0.23106 0.22649 0.090005"
-      rpy="0 0 0" />
-    <parent
-      link="x650_0/base_link" />
-    <child
-      link="x650_0/front_prop_cw_link" />
-    <axis
-      xyz="0 0 1" />
-    <limit effort="1e12" velocity="1e12"/>
-    <dynamics damping="0.0" friction="0.0"/>
-  </joint>
-  <link
-    name="x650_0/back_prop_ccw_link">
-    <inertial>
-      <origin
-        xyz="1.92448384979671E-05 -0.000547906471534965 0.00827249285044868"
-        rpy="0 0 0" />
-      <mass
-        value="0.0232876035112873" />
-      <inertia
-        ixx="7.81282403750946E-07"
-        ixy="-1.92967614763292E-06"
-        ixz="-5.83954145488408E-08"
-        iyy="2.83627824183673E-05"
-        iyz="-3.95754090522907E-08"
-        izz="2.90934055502375E-05" />
-    </inertial>
-    <visual>
-      <origin
-        xyz="0 0 0"
-        rpy="0 0 0" />
-      <geometry>
-        <mesh
-          filename="file://$(find uav_description)/meshes/back_prop_ccw_link.STL" />
-      </geometry>
-      <material
-        name="">
-        <color
-          rgba="0.752941176470588 0.752941176470588 0.752941176470588 1" />
-      </material>
-    </visual>
-    <collision>
-      <origin
-        xyz="0 0 0"
-        rpy="0 0 0" />
-      <geometry>
-        <mesh
-          filename="file://$(find uav_description)/meshes/back_prop_ccw_link.STL" />
-      </geometry>
-    </collision>
-  </link>
-  <joint
-    name="x650_0/back_prop_ccw_joint"
-    type="continuous">
-    <origin
-      xyz="-0.2287 0.23276 0.086501"
-      rpy="0 0 0" />
-    <parent
-      link="x650_0/base_link" />
-    <child
-      link="x650_0/back_prop_ccw_link" />
-    <axis
-      xyz="0 0 1" />
-    <limit effort="1e12" velocity="1e12"/>
-    <dynamics damping="0.0" friction="0.0"/>
-  </joint>
-  <link
-    name="x650_0/back_prop_cw_link">
-    <inertial>
-      <origin
-        xyz="2.5989393493131E-06 -0.00013126973913305 0.00575531220060893"
-        rpy="0 0 0" />
-      <mass
-        value="0.0232866239768517" />
-      <inertia
-        ixx="6.48789609174199E-07"
-        ixy="-1.71375304374027E-07"
-        ixz="1.27526457477932E-10"
-        iyy="2.84774113589609E-05"
-        iyz="5.48167333347854E-11"
-        izz="2.90799957464871E-05" />
-    </inertial>
-    <visual>
-      <origin
-        xyz="0 0 0"
-        rpy="0 0 0" />
-      <geometry>
-        <mesh
-          filename="file://$(find uav_description)/meshes/back_prop_cw_link.STL" />
-      </geometry>
-      <material
-        name="">
-        <color
-          rgba="0.752941176470588 0.752941176470588 0.752941176470588 1" />
-      </material>
-    </visual>
-    <collision>
-      <origin
-        xyz="0 0 0"
-        rpy="0 0 0" />
-      <geometry>
-        <mesh
-          filename="file://$(find uav_description)/meshes/back_prop_cw_link.STL" />
-      </geometry>
-    </collision>
-  </link>
-  <joint
-    name="x650_0/back_prop_cw_joint"
-    type="continuous">
-    <origin
-      xyz="-0.23496 -0.22701 0.086701"
-      rpy="0 0 0" />
-    <parent
-      link="x650_0/base_link" />
-    <child
-      link="x650_0/back_prop_cw_link" />
-    <axis
-      xyz="0 0 1" />
-    <limit effort="1e12" velocity="1e12"/>
-    <dynamics damping="0.0" friction="0.0"/>
-  </joint>
-  <link
-    name="x650_0/depth_camera_link">
-    <inertial>
-      <origin
-        xyz="0.0149830161779797 -6.98368398157727E-05 9.2241584007894E-06"
-        rpy="0 0 0" />
-      <mass
-        value="0.0907155514174442" />
+  <link name="base_link">
+    <inertial>
+      <origin xyz="-0.0025838 0.00051225 -0.019551" rpy="0 0 0" />
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