Commit message: Colors for Gazebo and RViz added.

File: src/uav_description/urdf/uav.gazebo.xacro (robot description, xacro)
@@ -1,17 +1,89 @@
 <?xml version="1.0"?>
 <robot name="uav_uav" xmlns:xacro="http://ros.org/wiki/xacro">
-    <!-- Color definitions-->
-    <xacro:property name="prop_color" value="Gazebo/Black" />
-    <xacro:property name="rgbd_cam_color" value="Gazebo/White" />
-    <xacro:property name="lidar_color" value="Gazebo/Black" />
-    <!-- Propellers -->
+    <gazebo reference="back_prop_cw_link">
+        <material>${gazebo_black}</material>
+        <mu1>0.1</mu1>
+        <mu2>0.1</mu2>
+        <gravity>true</gravity>
+    </gazebo>
+    <gazebo reference="back_prop_ccw_link">
+        <material>${gazebo_black}</material>
+        <mu1>0.1</mu1>
+        <mu2>0.1</mu2>
+        <gravity>true</gravity>
+    </gazebo>
+    <!-- Base link -->
+    <gazebo reference="base_link">
+        <material>${gazebo_grey}</material>
+        <mu1>0.1</mu1>
+        <mu2>0.1</mu2>
+        <gravity>true</gravity>
+    </gazebo>
+    <!-- Front CCW -->
+    <gazebo reference="front_arm_ccw_link">
+        <material>${gazebo_grey}</material>
+        <mu1>0.1</mu1>
+        <mu2>0.1</mu2>
+        <gravity>true</gravity>
+    </gazebo>
+    <gazebo reference="front_motor_ccw_link">
+        <material>${gazebo_grey}</material>
+        <mu1>0.1</mu1>
+        <mu2>0.1</mu2>
+        <gravity>true</gravity>
+    </gazebo>
+    <gazebo reference="front_prop_ccw_link">
+        <material>${gazebo_black}</material>
+        <mu1>0.1</mu1>
+        <mu2>0.1</mu2>
+        <gravity>true</gravity>
+    </gazebo>
+    <!-- Front CW -->
+    <gazebo reference="front_arm_cw_link">
+        <material>${gazebo_grey}</material>
+        <mu1>0.1</mu1>
+        <mu2>0.1</mu2>
+        <gravity>true</gravity>
+    </gazebo>
+    <gazebo reference="front_motor_cw_link">
+        <material>${gazebo_dark_grey}</material>
+        <mu1>0.1</mu1>
+        <mu2>0.1</mu2>
+        <gravity>true</gravity>
+    </gazebo>
     <gazebo reference="front_prop_cw_link">
-        <material>${prop_color}</material>
-        <mu1>0.1</mu1>
-        <mu2>0.1</mu2>
-        <gravity>true</gravity>
-    </gazebo>
-    <gazebo reference="front_prop_ccw_link">
-        <material>${prop_color}</material>
+        <material>${gazebo_black}</material>
+        <mu1>0.1</mu1>
+        <mu2>0.1</mu2>
+        <gravity>true</gravity>
+    </gazebo>
+    <!-- Back CCW -->
+    <gazebo reference="back_arm_ccw_link">
+        <material>${gazebo_grey}</material>
+        <mu1>0.1</mu1>
+        <mu2>0.1</mu2>
+        <gravity>true</gravity>
+    </gazebo>
+    <gazebo reference="back_motor_ccw_link">
+        <material>${gazebo_dark_grey}</material>
+        <mu1>0.1</mu1>
+        <mu2>0.1</mu2>
+        <gravity>true</gravity>
+    </gazebo>
+    <gazebo reference="back_prop_ccw_link">
+        <material>${gazebo_black}</material>
+        <mu1>0.1</mu1>
+        <mu2>0.1</mu2>
+        <gravity>true</gravity>
+    </gazebo>
+    <!-- Back CW -->
+    <gazebo reference="back_arm_cw_link">
+        <material>${gazebo_dark_grey}</material>
+        <mu1>0.1</mu1>
+        <mu2>0.1</mu2>
+        <gravity>true</gravity>
+    </gazebo>
+    <gazebo reference="back_motor_cw_link">
+        <material>${gazebo_dark_grey}</material>
         <mu1>0.1</mu1>
         <mu2>0.1</mu2>
@@ -19,11 +91,40 @@
     </gazebo>
     <gazebo reference="back_prop_cw_link">
-        <material>${prop_color}</material>
-        <mu1>0.1</mu1>
-        <mu2>0.1</mu2>
-        <gravity>true</gravity>
-    </gazebo>
-    <gazebo reference="back_prop_ccw_link">
-        <material>${prop_color}</material>
+        <material>${gazebo_black}</material>
+        <mu1>0.1</mu1>
+        <mu2>0.1</mu2>
+        <gravity>true</gravity>
+    </gazebo>
+    <!-- Telemetry -->
+    <gazebo reference="telemetry_link">
+        <material>${gazebo_black}</material>
+        <mu1>0.1</mu1>
+        <mu2>0.1</mu2>
+        <gravity>true</gravity>
+    </gazebo>
+    <!-- GPS module -->
+    <gazebo reference="gps_module_link">
+        <material>${gazebo_black}</material>
+        <mu1>0.1</mu1>
+        <mu2>0.1</mu2>
+        <gravity>true</gravity>
+    </gazebo>
+    <!-- Pixhawk Jetson Nanon microcontroller -->
+    <gazebo reference="pixhawk_jetson_mc_link">
+        <material>${gazebo_gazebo_flatblack}</material>
+        <mu1>0.1</mu1>
+        <mu2>0.1</mu2>
+        <gravity>true</gravity>
+    </gazebo>
+    <!-- Left landing gear -->
+    <gazebo reference="left_landing_gear_link">
+        <material>${gazebo_gazebo_flatblack}</material>
+        <mu1>0.1</mu1>
+        <mu2>0.1</mu2>
+        <gravity>true</gravity>
+    </gazebo>
+    <!-- Right landing gear -->
+    <gazebo reference="right_landing_gear_link">
+        <material>${gazebo_gazebo_flatblack}</material>
         <mu1>0.1</mu1>
         <mu2>0.1</mu2>
@@ -32,5 +133,5 @@
     <!-- Depth camera -->
     <gazebo reference="depth_camera_link">
-        <material>${rgbd_cam_color}</material>
+        <material>${gazebo_white}</material>
         <mu1>0.1</mu1>
         <mu2>0.1</mu2>
@@ -57,5 +158,5 @@
     <!-- Lidar sensor -->
     <gazebo reference="lidar_link">
-        <material>${lidar_color}</material>
+        <material>${gazebo_dark_grey}</material>
         <mu1>0.1</mu1>
         <mu2>0.1</mu2>

File: src/uav_description/urdf/uav.urdf.xacro (robot description, xacro)
@@ -4,4 +4,5 @@
      For more information, please see http://wiki.ros.org/sw_urdf_exporter -->
 <robot name="uav_uav" xmlns:xacro="http://www.ros.org/wiki/xacro">
+  <xacro:include filename="$(find uav_description)/urdf/core.xacro"/>
   <xacro:include filename="$(find uav_description)/urdf/uav.gazebo.xacro"/>
   <link name="base_link">
@@ -155,7 +156,7 @@
         <mesh filename="file://$(find uav_description)/meshes/front_arm_cw_link.STL" />
       </geometry>
-      <material name="">
-        <color rgba="0.529411764705882 0.549019607843137 0.549019607843137 1" />
-      </material>
+      <material name="dark_gray" />
+        <!-- <color rgba="0.529411764705882 0.549019607843137 0.549019607843137 1" /> -->
+      <!-- </material> -->
     </visual>
     <collision>

Commit message: Lidar sensor added, lidar sensor data shown in RViz.

File: src/uav_description/urdf/uav.gazebo.xacro (robot description, xacro)
@@ -141,15 +141,16 @@
                 <horizontal_fov>1.5184</horizontal_fov>
                 <image>
-                    <width>424</width>
-                    <height>240</height>
+                    <width>600</width>
+                    <height>480</height>
+                    <format>RGB_INT8</format>
                 </image>
                 <clip>
-                    <near>0.05</near>
-                    <far>1.5</far>
+                    <near>0.6</near>
+                    <far>6.0</far>
                 </clip>
             </camera>
             <always_on>1</always_on>
             <gz_frame_id>depth_camera_link</gz_frame_id>
-            <topic>cam_1</topic>
+            <topic>camera</topic>
             <update_rate>15.0</update_rate>
             <visualize>true</visualize>
@@ -168,8 +169,10 @@
             <always_on>true</always_on>
             <visualize>true</visualize>
+            <gz_frame_id>lidar_link</gz_frame_id>
             <lidar>
                 <scan>
                     <horizontal>
-                        <samples>720</samples>  <!-- TODO: Has to be adjusted -->
+                        <!-- Based on technical specs -->
+                        <samples>720</samples>
                         <resolution>1</resolution>
                         <min_angle>-3.14159</min_angle>
@@ -191,11 +194,22 @@
                 </scan>
                 <range>
-                    <min>0.2</min>                  <!-- TODO: Has to be adjusted -->
-                    <max>25.0</max>                 <!-- TODO: Has to be adjusted -->
-                    <resolution>0.225</resolution>  <!-- TODO: Has to be adjusted -->
+                    <min>0.15</min>
+                    <max>6.0</max>
+                    <resolution>0.001</resolution>
                 </range>
             </lidar>
-            <gz_frame_id>lidar_link</gz_frame_id>
         </sensor>
     </gazebo>
+    <gazebo>
+        <plugin filename="gz-sim-sensors-system" name="gz::sim::systems::Sensors">
+            <render_engine>ogre2</render_engine>
+        </plugin>
+    </gazebo>
+    <!-- Enables the communication with ros2_control -->
+    <!-- <gazebo>
+        <plugin name="gz_ros2_control::GazeboSimROS2ControlPlugin" filename="libgz_ros2_control-system.so">
+            <parameters>$(find hospibot_bringup)/config/controllers.yaml</parameters>
+            <controller_manager_node_name>controller_manager</controller_manager_node_name>
+        </plugin>
+    </gazebo> -->
 </robot>

File: src/uav_description/urdf/uav.urdf.xacro (robot description, xacro)
@@ -135,7 +135,6 @@
     <child link="front_prop_ccw_link" />
     <axis xyz="0 0 1" />
-    <limit
-      effort="100"
-      velocity="100" />
+    <limit effort="100" velocity="100" />
+    <dynamics damping="0.01" friction="0.0"/>
   </joint>
   <link name="front_arm_cw_link">
@@ -240,7 +239,6 @@
     <child link="front_prop_cw_link" />
     <axis xyz="0 0 1" />
-    <limit
-      effort="100"
-      velocity="100" />
+    <limit effort="100" velocity="100" />
+    <dynamics damping="0.01" friction="0.0"/>
   </joint>
   <link name="back_arm_ccw_link">
@@ -345,7 +343,6 @@
     <child link="back_prop_ccw_link" />
     <axis xyz="0 0 1" />
-    <limit
-      effort="100"
-      velocity="100" />
+    <limit effort="100" velocity="100" />
+    <dynamics damping="0.01" friction="0.0"/>
   </joint>
   <link name="back_arm_cw_link">
@@ -450,7 +447,6 @@
     <child link="back_prop_cw_link" />
     <axis xyz="0 0 1" />
-    <limit
-      effort="100"
-      velocity="100" />
+    <limit effort="100" velocity="100" />
+    <dynamics damping="0.01" friction="0.0"/>
   </joint>
   <link name="depth_camera_link">
