Commit message: UAV 3D model refactored and URDF file adjusted accordingly.

File: src/uav_description/urdf/uav.gazebo.xacro (robot description, xacro)
@@ -21,16 +21,4 @@
     </gazebo>
     <!-- Front CCW -->
-    <gazebo reference="front_arm_ccw_link">
-        <material>${gazebo_grey}</material>
-        <mu1>0.1</mu1>
-        <mu2>0.1</mu2>
-        <gravity>true</gravity>
-    </gazebo>
-    <gazebo reference="front_motor_ccw_link">
-        <material>${gazebo_grey}</material>
-        <mu1>0.1</mu1>
-        <mu2>0.1</mu2>
-        <gravity>true</gravity>
-    </gazebo>
     <gazebo reference="front_prop_ccw_link">
         <material>${gazebo_black}</material>
@@ -40,16 +28,4 @@
     </gazebo>
     <!-- Front CW -->
-    <gazebo reference="front_arm_cw_link">
-        <material>${gazebo_grey}</material>
-        <mu1>0.1</mu1>
-        <mu2>0.1</mu2>
-        <gravity>true</gravity>
-    </gazebo>
-    <gazebo reference="front_motor_cw_link">
-        <material>${gazebo_dark_grey}</material>
-        <mu1>0.1</mu1>
-        <mu2>0.1</mu2>
-        <gravity>true</gravity>
-    </gazebo>
     <gazebo reference="front_prop_cw_link">
         <material>${gazebo_black}</material>
@@ -59,16 +35,4 @@
     </gazebo>
     <!-- Back CCW -->
-    <gazebo reference="back_arm_ccw_link">
-        <material>${gazebo_grey}</material>
-        <mu1>0.1</mu1>
-        <mu2>0.1</mu2>
-        <gravity>true</gravity>
-    </gazebo>
-    <gazebo reference="back_motor_ccw_link">
-        <material>${gazebo_dark_grey}</material>
-        <mu1>0.1</mu1>
-        <mu2>0.1</mu2>
-        <gravity>true</gravity>
-    </gazebo>
     <gazebo reference="back_prop_ccw_link">
         <material>${gazebo_black}</material>
@@ -78,24 +42,5 @@
     </gazebo>
     <!-- Back CW -->
-    <gazebo reference="back_arm_cw_link">
-        <material>${gazebo_dark_grey}</material>
-        <mu1>0.1</mu1>
-        <mu2>0.1</mu2>
-        <gravity>true</gravity>
-    </gazebo>
-    <gazebo reference="back_motor_cw_link">
-        <material>${gazebo_dark_grey}</material>
-        <mu1>0.1</mu1>
-        <mu2>0.1</mu2>
-        <gravity>true</gravity>
-    </gazebo>
     <gazebo reference="back_prop_cw_link">
-        <material>${gazebo_black}</material>
-        <mu1>0.1</mu1>
-        <mu2>0.1</mu2>
-        <gravity>true</gravity>
-    </gazebo>
-    <!-- Telemetry -->
-    <gazebo reference="telemetry_link">
         <material>${gazebo_black}</material>
         <mu1>0.1</mu1>
@@ -106,25 +51,4 @@
     <gazebo reference="gps_module_link">
         <material>${gazebo_black}</material>
-        <mu1>0.1</mu1>
-        <mu2>0.1</mu2>
-        <gravity>true</gravity>
-    </gazebo>
-    <!-- Pixhawk Jetson Nanon microcontroller -->
-    <gazebo reference="pixhawk_jetson_mc_link">
-        <material>${gazebo_gazebo_flatblack}</material>
-        <mu1>0.1</mu1>
-        <mu2>0.1</mu2>
-        <gravity>true</gravity>
-    </gazebo>
-    <!-- Left landing gear -->
-    <gazebo reference="left_landing_gear_link">
-        <material>${gazebo_gazebo_flatblack}</material>
-        <mu1>0.1</mu1>
-        <mu2>0.1</mu2>
-        <gravity>true</gravity>
-    </gazebo>
-    <!-- Right landing gear -->
-    <gazebo reference="right_landing_gear_link">
-        <material>${gazebo_gazebo_flatblack}</material>
         <mu1>0.1</mu1>
         <mu2>0.1</mu2>

File: src/uav_description/urdf/uav.urdf.xacro (robot description, xacro)
@@ -3,688 +3,426 @@
      Commit Version: 1.6.0-4-g7f85cfe  Build Version: 1.6.7995.38578
      For more information, please see http://wiki.ros.org/sw_urdf_exporter -->
-<robot name="uav_uav" xmlns:xacro="http://www.ros.org/wiki/xacro">
+<robot name="UAV_X650" xmlns:xacro="http://www.ros.org/wiki/xacro">
   <xacro:include filename="$(find uav_description)/urdf/core.xacro"/>
   <xacro:include filename="$(find uav_description)/urdf/uav.gazebo.xacro"/>
   <link name="base_link">
     <inertial>
-      <origin xyz="-0.0025838 0.00051225 -0.019551" rpy="0 0 0" />
-      <mass value="1.4371" />
-      <inertia
-        ixx="0.00098413"
-        ixy="4.9253E-05"
-        ixz="6.648E-07"
-        iyy="0.0038692"
-        iyz="2.8305E-08"
-        izz="0.0047748" />
+      <origin
+        xyz="-0.00372276524577257 -0.00744305903269664 8.57191257253331E-05"
+        rpy="0 0 0" />
+      <mass
+        value="2.79538458384779" />
+      <inertia
+        ixx="0.00251955261705473"
+        ixy="-1.69520154890596E-05"
+        ixz="-9.26102151476342E-05"
+        iyy="0.00725324885475083"
+        iyz="5.60750810648567E-06"
+        izz="0.00570366183964889" />
     </inertial>
     <visual>
       <origin xyz="0 0 0" rpy="0 0 0" />
       <geometry>
-        <mesh filename="file://$(find uav_description)/meshes/base_link.STL" />
-      </geometry>
-      <material name="">
-        <color rgba="0.75294 0.75294 0.75294 1" />
-      </material>
-    </visual>
-    <collision>
-      <origin xyz="0 0 0" rpy="0 0 0" />
-      <geometry>
-        <mesh filename="file://$(find uav_description)/meshes/base_link.STL" />
-      </geometry>
-    </collision>
-  </link>
-  <link name="front_arm_ccw_link">
-    <inertial>
-      <origin xyz="5.14187352146367E-06 0.000103088445734027 0.101201605126024" rpy="0 0 0" />
-      <mass value="0.163581488184572" />
-      <inertia
-        ixx="0.000495858318312467"
-        ixy="1.69719015225508E-08"
-        ixz="-1.5555901263121E-08"
-        iyy="0.000496622426658751"
-        iyz="3.01279610270572E-08"
-        izz="1.58530814438199E-05" />
-    </inertial>
-    <visual>
-      <origin xyz="0 0 0" rpy="0 0 0" />
-      <geometry>
-        <mesh filename="file://$(find uav_description)/meshes/front_arm_ccw_link.STL" />
-      </geometry>
-      <material name="">
-        <color rgba="0.529411764705882 0.549019607843137 0.549019607843137 1" />
-      </material>
-    </visual>
-    <collision>
-      <origin xyz="0 0 0" rpy="0 0 0" />
-      <geometry>
-        <mesh filename="file://$(find uav_description)/meshes/front_arm_ccw_link.STL" />
-      </geometry>
-    </collision>
-  </link>
-  <joint name="front_arm_ccw_joint" type="fixed">
-    <origin xyz="0.080474 -0.082381 0.043625" rpy="-1.5708 0 -2.3562" />
-    <parent link="base_link" />
-    <child link="front_arm_ccw_link" />
-    <axis xyz="0 0 0" />
-  </joint>
-  <link name="front_motor_ccw_link">
-    <inertial>
-      <origin xyz="-5.94792757824258E-08 0.0089323100189773 0.000144520880497323" rpy="0 0 0" />
-      <mass value="0.107028077375073" />
-      <inertia
-        ixx="1.99852843592467E-05"
-        ixy="-9.14808285986034E-11"
-        ixz="-2.70349866236598E-09"
-        iyy="2.60832369889382E-05"
-        iyz="2.20707374208015E-07"
-        izz="1.97284529490253E-05" />
-    </inertial>
-    <visual>
-      <origin xyz="0 0 0" rpy="0 0 0" />
-      <geometry>
-        <mesh filename="file://$(find uav_description)/meshes/front_motor_ccw_link.STL" />
-      </geometry>
-      <material name="">
-        <color rgba="0.898039215686275 0.917647058823529 0.929411764705882 1" />
-      </material>
-    </visual>
-    <collision>
-      <origin xyz="0 0 0" rpy="0 0 0" />
-      <geometry>
-        <mesh filename="file://$(find uav_description)/meshes/front_motor_ccw_link.STL" />
-      </geometry>
-    </collision>
-  </link>
-  <joint name="front_motor_ccw_joint" type="fixed">
-    <origin xyz="0 -0.022 0.209" rpy="0 0 3.1416" />
-    <parent link="front_arm_ccw_link" />
-    <child link="front_motor_ccw_link" />
-    <axis xyz="0 0 0" />
-  </joint>
-  <link name="front_prop_ccw_link">
-    <inertial>
-      <origin xyz="2.11228381036821E-05 -0.000575623595751584 0.00874250262086616" rpy="0 0 0" />
-      <mass value="0.0232885965258771" />
-      <inertia
-        ixx="7.81406911098823E-07"
-        ixy="-1.93046094872738E-06"
-        ixz="-5.84228099790564E-08"
-        iyy="2.83657143471591E-05"
-        iyz="-3.95826230995061E-08"
-        izz="2.90964600411815E-05" />
-    </inertial>
-    <visual>
-      <origin xyz="0 0 0" rpy="0 0 0" />
-      <geometry>
-        <mesh filename="file://$(find uav_description)/meshes/front_prop_ccw_link.STL" />
-      </geometry>
-      <material name="">
-        <color rgba="0.752941176470588 0.752941176470588 0.752941176470588 1" />
-      </material>
-    </visual>
-    <collision>
-      <origin xyz="0 0 0" rpy="0 0 0" />
-      <geometry>
-        <mesh filename="file://$(find uav_description)/meshes/front_prop_ccw_link.STL" />
-      </geometry>
-    </collision>
-  </link>
-  <joint name="front_prop_ccw_joint" type="continuous">
-    <origin xyz="0 0.024318 0" rpy="1.5108 0.40362 3.1394" />
-    <parent link="front_motor_ccw_link" />
-    <child link="front_prop_ccw_link" />
-    <axis xyz="0 0 1" />
-    <limit effort="100" velocity="100" />
-    <dynamics damping="0.01" friction="0.0"/>
-  </joint>
-  <link name="front_arm_cw_link">
-    <inertial>
-      <origin xyz="5.14187362136292E-06 0.000103088445712607 0.10120160512516" rpy="0 0 0" />
-      <mass value="0.163581488183559" />
-      <inertia
-        ixx="0.000495858318312464"
-        ixy="1.69719015255707E-08"
-        ixz="-1.55559012619851E-08"
-        iyy="0.000496622426658752"
-        iyz="3.01279610276289E-08"
-        izz="1.58530814438145E-05" />
-    </inertial>
-    <visual>
-      <origin xyz="0 0 0" rpy="0 0 0" />
-      <geometry>
-        <mesh filename="file://$(find uav_description)/meshes/front_arm_cw_link.STL" />
-      </geometry>
-      <material name="dark_gray" />
-        <!-- <color rgba="0.529411764705882 0.549019607843137 0.549019607843137 1" /> -->
-      <!-- </material> -->
-    </visual>
-    <collision>
-      <origin xyz="0 0 0" rpy="0 0 0" />
-      <geometry>
-        <mesh filename="file://$(find uav_description)/meshes/front_arm_cw_link.STL" />
-      </geometry>
-    </collision>
-  </link>
-  <joint name="front_arm_cw_joint" type="fixed">
-    <origin xyz="0.0804741042413417 0.0818613658673572 0.0436254108086869" rpy="-1.5707963267949 0 -0.785398163397448" />
-    <parent link="base_link" />
-    <child link="front_arm_cw_link" />
-    <axis xyz="0 0 0" />
-  </joint>
-  <link name="front_motor_cw_link">
-    <inertial>
-      <origin xyz="-5.94792757269147E-08 0.00893231001897728 0.000144520880497323" rpy="0 0 0" />
-      <mass value="0.107028077375073" />
-      <inertia
-        ixx="1.99852843592467E-05"
-        ixy="-9.14808285889419E-11"
-        ixz="-2.70349866238292E-09"
-        iyy="2.60832369889382E-05"
-        iyz="2.20707374208015E-07"
-        izz="1.97284529490253E-05" />
-    </inertial>
-    <visual>
-      <origin xyz="0 0 0" rpy="0 0 0" />
-      <geometry>
-        <mesh filename="file://$(find uav_description)/meshes/front_motor_cw_link.STL" />
-      </geometry>
-      <material name="">
-        <color rgba="0.898039215686275 0.917647058823529 0.929411764705882 1" />
-      </material>
-    </visual>
-    <collision>
-      <origin xyz="0 0 0" rpy="0 0 0" />
-      <geometry>
-        <mesh filename="file://$(find uav_description)/meshes/front_motor_cw_link.STL" />
-      </geometry>
-    </collision>
-  </link>
-  <joint name="front_motor_cw_joint" type="fixed">
-    <origin xyz="0 -0.022 0.209" rpy="0 0 3.14159265358979" />
-    <parent link="front_arm_cw_link" />
-    <child link="front_motor_cw_link" />
-    <axis xyz="0 0 0" />
-  </joint>
-  <link name="front_prop_cw_link">
-    <inertial>
-      <origin xyz="1.70322207349027E-06 -0.000131171076623415 0.00551466266249338" rpy="0 0 0" />
-      <mass value="0.023286089430334" />
-      <inertia
-        ixx="6.48766355495004E-07"
-        ixy="-1.71425530770085E-07"
-        ixz="1.31741915464193E-10"
-        iyy="2.84758053692334E-05"
-        iyz="5.4172324392471E-11"
-        izz="2.90783664832776E-05" />
-    </inertial>
-    <visual>
-      <origin xyz="0 0 0" rpy="0 0 0" />
-      <geometry>
-        <mesh filename="file://$(find uav_description)/meshes/front_prop_cw_link.STL" />
-      </geometry>
-      <material name="">
-        <color rgba="0.752941176470588 0.752941176470588 0.752941176470588 1" />
-      </material>
-    </visual>
-    <collision>
-      <origin xyz="0 0 0" rpy="0 0 0" />
-      <geometry>
-        <mesh filename="file://$(find uav_description)/meshes/front_prop_cw_link.STL" />
-      </geometry>
-    </collision>
-  </link>
-  <joint name="front_prop_cw_joint" type="continuous">
-    <origin xyz="0 0.027 0" rpy="-1.5708 0.94181 0" />
-    <parent link="front_motor_cw_link" />
-    <child link="front_prop_cw_link" />
-    <axis xyz="0 0 1" />
-    <limit effort="100" velocity="100" />
-    <dynamics damping="0.01" friction="0.0"/>
-  </joint>
-  <link name="back_arm_ccw_link">
-    <inertial>
-      <origin xyz="5.1418737516476E-06 0.000103088445681951 0.101201605122122" rpy="0 0 0" />
-      <mass value="0.163581488181259" />
-      <inertia
-        ixx="0.000495858318312453"
-        ixy="1.69719015333838E-08"
-        ixz="-1.55559012587393E-08"
-        iyy="0.000496622426658752"
-        iyz="3.01279610291379E-08"
-        izz="1.58530814438022E-05" />
-    </inertial>
-    <visual>
-      <origin xyz="0 0 0" rpy="0 0 0" />
-      <geometry>
-        <mesh filename="file://$(find uav_description)/meshes/back_arm_ccw_link.STL" />
-      </geometry>
-      <material name="">
-        <color rgba="0.529411764705882 0.549019607843137 0.549019607843137 1" />
-      </material>
-    </visual>
-    <collision>
-      <origin xyz="0 0 0" rpy="0 0 0" />
-      <geometry>
-        <mesh filename="file://$(find uav_description)/meshes/back_arm_ccw_link.STL" />
-      </geometry>
-    </collision>
-  </link>
-  <joint name="back_arm_ccw_joint" type="fixed">
-    <origin xyz="-0.0837685364457783 0.0818613658673572 0.0436254108086869" rpy="-1.5707963267949 0 0.785398163397448" />
-    <parent link="base_link" />
-    <child link="back_arm_ccw_link" />
-    <axis xyz="0 0 0" />
-  </joint>
-  <link name="back_motor_ccw_link">
-    <inertial>
-      <origin xyz="-5.94792757546703E-08 0.00893231001897728 0.000144520880497268" rpy="0 0 0" />
-      <mass value="0.107028077375073" />
-      <inertia
-        ixx="1.99852843592467E-05"
-        ixy="-9.14808285776261E-11"
-        ixz="-2.70349866238376E-09"
-        iyy="2.60832369889382E-05"
-        iyz="2.20707374208025E-07"
-        izz="1.97284529490253E-05" />
-    </inertial>
-    <visual>
-      <origin xyz="0 0 0" rpy="0 0 0" />
-      <geometry>
-        <mesh filename="file://$(find uav_description)/meshes/back_motor_ccw_link.STL" />
-      </geometry>
-      <material name="">
-        <color rgba="0.898039215686275 0.917647058823529 0.929411764705882 1" />
-      </material>
-    </visual>
-    <collision>
-      <origin xyz="0 0 0" rpy="0 0 0" />
-      <geometry>
-        <mesh filename="file://$(find uav_description)/meshes/back_motor_ccw_link.STL" />
-      </geometry>
-    </collision>
-  </link>
-  <joint name="back_motor_ccw_joint" type="fixed">
-    <origin xyz="0 -0.022 0.209" rpy="0 0 3.14159265358979" />
-    <parent link="back_arm_ccw_link" />
-    <child link="back_motor_ccw_link" />
-    <axis xyz="0 0 0" />
-  </joint>
-  <link name="back_prop_ccw_link">
-    <inertial>
-      <origin xyz="2.11084475078838E-05 -0.000575616574168103 0.00874246753673161" rpy="0 0 0" />
-      <mass value="0.0232874208355566" />
-      <inertia
-        ixx="7.81255330319095E-07"
-        ixy="-1.92969901663437E-06"
-        ixz="-5.83835421242838E-08"
-        iyy="2.83627343839516E-05"
-        iyz="-3.95752885069779E-08"
-        izz="2.90933307991966E-05" />
-    </inertial>
-    <visual>
-      <origin xyz="0 0 0" rpy="0 0 0" />
-      <geometry>
-        <mesh filename="file://$(find uav_description)/meshes/back_prop_ccw_link.STL" />
-      </geometry>
-      <material name="">
-        <color rgba="0.752941176470588 0.752941176470588 0.752941176470588 1" />
-      </material>
-    </visual>
-    <collision>
-      <origin xyz="0 0 0" rpy="0 0 0" />
-      <geometry>
-        <mesh filename="file://$(find uav_description)/meshes/back_prop_ccw_link.STL" />
-      </geometry>
-    </collision>
-  </link>
-  <joint name="back_prop_ccw_joint" type="continuous">
-    <origin xyz="0 0.024318 0" rpy="-1.6317 -0.71466 0.0026132" />
-    <parent link="back_motor_ccw_link" />
-    <child link="back_prop_ccw_link" />
-    <axis xyz="0 0 1" />
-    <limit effort="100" velocity="100" />
-    <dynamics damping="0.01" friction="0.0"/>
-  </joint>
-  <link name="back_arm_cw_link">
-    <inertial>
-      <origin xyz="5.14187358731377E-06 0.000103088445712947 0.101201605123568" rpy="0 0 0" />
-      <mass value="0.163581488182937" />
-      <inertia
-        ixx="0.000495858318312459"
-        ixy="1.69719015281368E-08"
-        ixz="-1.555590126059E-08"
-        iyy="0.000496622426658752"
-        iyz="3.01279610281771E-08"
-        izz="1.58530814438118E-05" />
-    </inertial>
-    <visual>
-      <origin xyz="0 0 0" rpy="0 0 0" />
-      <geometry>
-        <mesh filename="file://$(find uav_description)/meshes/back_arm_cw_link.STL" />
-      </geometry>
-      <material name="">
-        <color rgba="0.529411764705882 0.549019607843137 0.549019607843137 1" />
-      </material>
-    </visual>
-    <collision>
-      <origin xyz="0 0 0" rpy="0 0 0" />
-      <geometry>
-        <mesh filename="file://$(find uav_description)/meshes/back_arm_cw_link.STL" />
-      </geometry>
-    </collision>
-  </link>
-  <joint name="back_arm_cw_joint" type="fixed">
-    <origin xyz="-0.0837685364457783 -0.0823812748197628 0.0436254108086869" rpy="-1.5707963267949 0 2.35619449019234" />
-    <parent link="base_link" />
-    <child link="back_arm_cw_link" />
-    <axis xyz="0 0 0" />
-  </joint>
-  <link name="back_motor_cw_link">
-    <inertial>
-      <origin xyz="-5.94792757269147E-08 0.0089323100189773 0.000144520880497323" rpy="0 0 0" />
-      <mass value="0.107028077375073" />
-      <inertia
-        ixx="1.99852843592466E-05"
-        ixy="-9.14808285823906E-11"
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
Commit message: ROS2 Controll implemented (not working at present) and ros_bridge yaml file modified.

File: src/uav_description/urdf/uav.gazebo.xacro (robot description, xacro)
@@ -1,16 +1,4 @@
 <?xml version="1.0"?>
 <robot name="uav_uav" xmlns:xacro="http://ros.org/wiki/xacro">
-    <gazebo reference="back_prop_cw_link">
-        <material>${gazebo_black}</material>
-        <mu1>0.1</mu1>
-        <mu2>0.1</mu2>
-        <gravity>true</gravity>
-    </gazebo>
-    <gazebo reference="back_prop_ccw_link">
-        <material>${gazebo_black}</material>
-        <mu1>0.1</mu1>
-        <mu2>0.1</mu2>
-        <gravity>true</gravity>
-    </gazebo>
     <!-- Base link -->
     <gazebo reference="base_link">
@@ -125,4 +113,5 @@
         </sensor>
     </gazebo>
+    <!-- Plugin for sensor handling -->
     <gazebo>
         <plugin filename="gz-sim-sensors-system" name="gz::sim::systems::Sensors">
@@ -131,9 +120,9 @@
     </gazebo>
     <!-- Enables the communication with ros2_control -->
-    <!-- <gazebo>
+    <gazebo>
         <plugin name="gz_ros2_control::GazeboSimROS2ControlPlugin" filename="libgz_ros2_control-system.so">
-            <parameters>$(find hospibot_bringup)/config/controllers.yaml</parameters>
+            <parameters>$(find uav_bringup)/config/uav_controllers.yaml</parameters>
             <controller_manager_node_name>controller_manager</controller_manager_node_name>
         </plugin>
-    </gazebo> -->
+    </gazebo>
 </robot>

Commit message: Controllers with spawning delay added (because of loading time of Gazebo).

File: src/uav_description/urdf/uav.gazebo.xacro (robot description, xacro)
@@ -1,4 +1,4 @@
 <?xml version="1.0"?>
-<robot name="uav_uav" xmlns:xacro="http://ros.org/wiki/xacro">
+<robot name="uav" xmlns:xacro="http://ros.org/wiki/xacro">
     <!-- Base link -->
     <gazebo reference="base_link">
@@ -120,9 +120,9 @@
     </gazebo>
     <!-- Enables the communication with ros2_control -->
-    <!-- <gazebo>
-        <plugin name="gz_ros2_control::GazeboSimROS2ControlPlugin" filename="libgz_ros2_control-system.so">
-            <parameters>$(find uav_bringup)/config/uav_controllers.yaml</parameters>
-            <controller_manager_node_name>controller_manager</controller_manager_node_name>
+    <gazebo>
+        <plugin name="gz_ros2_control::GazeboSimROS2ControlPlugin" filename="gz_ros2_control-system">
+            <parameters>$(find uav_control)/config/uav_controllers.yaml</parameters>
+            <!-- <controller_manager_node_name>controller_manager</controller_manager_node_name> -->
         </plugin>
-    </gazebo> -->
+    </gazebo>
 </robot>

File: src/uav_description/urdf/uav.ros2_control.xacro (robot description, xacro)
@@ -1,3 +1,32 @@
 <?xml version="1.0"?>
-<robot name="uav_uav" xmlns:xacro="http://ros.org/wiki/xacro">
+<robot name="uav" xmlns:xacro="http://ros.org/wiki/xacro">
+    <ros2_control name="uav_hardware_interface" type="system">
+        <hardware>
+            <plugin>gz_ros2_control/GazeboSimSystem</plugin>
+        </hardware>
+        <joint name="front_prop_cw_joint">
+            <command_interface name="velocity"/>
+            <state_interface name="position"/>
+            <state_interface name="velocity"/>
+            <state_interface name="effort"/>
+        </joint>
+        <joint name="front_prop_ccw_joint">
+            <command_interface name="velocity"/>
+            <state_interface name="position"/>
+            <state_interface name="velocity"/>
+            <state_interface name="effort"/>
+        </joint>
+        <joint name="back_prop_cw_joint">
+            <command_interface name="velocity"/>
+            <state_interface name="position"/>
+            <state_interface name="velocity"/>
+            <state_interface name="effort"/>
+        </joint>
+        <joint name="back_prop_ccw_joint">
+            <command_interface name="velocity"/>
+            <state_interface name="position"/>
+            <state_interface name="velocity"/>
+            <state_interface name="effort"/>
+        </joint>
+    </ros2_control>
 </robot>

File: src/uav_description/urdf/uav.urdf.xacro (robot description, xacro)
@@ -7,4 +7,5 @@
   <xacro:include filename="$(find uav_description)/urdf/uav.gazebo.xacro"/>
   <xacro:include filename="$(find uav_description)/urdf/uav.ros2_control.xacro"/>
+  <link name="base_footprint"/>
   <link name="base_link">
     <inertial>
@@ -44,4 +45,10 @@
     </collision>
   </link>
+  <joint name="base_footprint_joint"
+    type="fixed">
+    <origin xyz="0 0 0" rpy="0 0 0" />
+    <parent link="base_footprint" />
+    <child link="base_link" />
+  </joint>
   <link
     name="lidar_link">
