Commit message: Motor controller plugins added and controller bug fixed.

File: src/uav_description/urdf/uav.gazebo.xacro (robot description, xacro)
@@ -123,6 +123,85 @@
         <plugin name="gz_ros2_control::GazeboSimROS2ControlPlugin" filename="gz_ros2_control-system">
             <parameters>$(find uav_control)/config/uav_controllers.yaml</parameters>
-            <!-- <controller_manager_node_name>controller_manager</controller_manager_node_name> -->
         </plugin>
     </gazebo>
+    <!-- Front CCW motor -->
+    <gazebo>
+      <plugin filename="gz-sim-multicopter-motor-model-system" name="gz::sim::systems::MulticopterMotorModel">
+        <jointName>front_prop_ccw_joint</jointName>
+        <linkName>front_prop_ccw_link</linkName>
+        <turningDirection>ccw</turningDirection>
+        <timeConstantUp>0.0125</timeConstantUp>
+        <timeConstantDown>0.025</timeConstantDown>
+        <maxRotVelocity>8000</maxRotVelocity>
+        <motorConstant>3.0e-05</motorConstant>
+        <momentConstant>0.016</momentConstant>
+        <commandSubTopic>gazebo/command/motor_speed</commandSubTopic>
+        <actuator_number>0</actuator_number>
+        <rotorDragCoefficient>8.06428e-05</rotorDragCoefficient>
+        <rollingMomentCoefficient>1e-06</rollingMomentCoefficient>
+        <motorSpeedPubTopic>motor_speed/0</motorSpeedPubTopic>
+        <rotorVelocitySlowdownSim>1</rotorVelocitySlowdownSim>
+        <motorType>velocity</motorType>
+      </plugin>
+    </gazebo>
+    <!-- Front CW motor -->
+    <gazebo>
+      <plugin filename="gz-sim-multicopter-motor-model-system" name="gz::sim::systems::MulticopterMotorModel">
+        <jointName>front_prop_cw_joint</jointName>
+        <linkName>front_prop_cw_link</linkName>
+        <turningDirection>cw</turningDirection>
+        <timeConstantUp>0.0125</timeConstantUp>
+        <timeConstantDown>0.025</timeConstantDown>
+        <maxRotVelocity>8000</maxRotVelocity>
+        <motorConstant>3.0e-05</motorConstant>
+        <momentConstant>0.016</momentConstant>
+        <commandSubTopic>gazebo/command/motor_speed</commandSubTopic>
+        <actuator_number>1</actuator_number>
+        <rotorDragCoefficient>8.06428e-05</rotorDragCoefficient>
+        <rollingMomentCoefficient>1e-06</rollingMomentCoefficient>
+        <motorSpeedPubTopic>motor_speed/1</motorSpeedPubTopic>
+        <rotorVelocitySlowdownSim>1</rotorVelocitySlowdownSim>
+        <motorType>velocity</motorType>
+      </plugin>
+    </gazebo>
+    <!-- Back CCW motor -->
+    <gazebo>
+      <plugin filename="gz-sim-multicopter-motor-model-system" name="gz::sim::systems::MulticopterMotorModel">
+        <jointName>back_prop_ccw_joint</jointName>
+        <linkName>back_prop_ccw_link</linkName>
+        <turningDirection>ccw</turningDirection>
+        <timeConstantUp>0.0125</timeConstantUp>
+        <timeConstantDown>0.025</timeConstantDown>
+        <maxRotVelocity>8000</maxRotVelocity>
+        <motorConstant>3.0e-05</motorConstant>
+        <momentConstant>0.016</momentConstant>
+        <commandSubTopic>gazebo/command/motor_speed</commandSubTopic>
+        <actuator_number>2</actuator_number>
+        <rotorDragCoefficient>8.06428e-05</rotorDragCoefficient>
+        <rollingMomentCoefficient>1e-06</rollingMomentCoefficient>
+        <motorSpeedPubTopic>motor_speed/2</motorSpeedPubTopic>
+        <rotorVelocitySlowdownSim>1</rotorVelocitySlowdownSim>
+        <motorType>velocity</motorType>
+      </plugin>
+    </gazebo>
+    <!-- Back CW motor -->
+    <gazebo>
+      <plugin filename="gz-sim-multicopter-motor-model-system" name="gz::sim::systems::MulticopterMotorModel">
+        <jointName>back_prop_cw_joint</jointName>
+        <linkName>back_prop_cw_link</linkName>
+        <turningDirection>cw</turningDirection>
+        <timeConstantUp>0.0125</timeConstantUp>
+        <timeConstantDown>0.025</timeConstantDown>
+        <maxRotVelocity>8000</maxRotVelocity>
+        <motorConstant>3.0e-05</motorConstant>
+        <momentConstant>0.016</momentConstant>
+        <commandSubTopic>gazebo/command/motor_speed</commandSubTopic>
+        <actuator_number>3</actuator_number>
+        <rotorDragCoefficient>8.06428e-05</rotorDragCoefficient>
+        <rollingMomentCoefficient>1e-06</rollingMomentCoefficient>
+        <motorSpeedPubTopic>motor_speed/3</motorSpeedPubTopic>
+        <rotorVelocitySlowdownSim>1</rotorVelocitySlowdownSim>
+        <motorType>velocity</motorType>
+      </plugin>
+    </gazebo>
 </robot>

File: src/uav_description/urdf/uav.urdf.xacro (robot description, xacro)
@@ -209,7 +209,6 @@
     <axis
       xyz="0 0 1" />
-    <limit
-      effort="100"
-      velocity="100" />
+    <limit effort="1000000" velocity="10000"/>
+    <dynamics damping="0.0" friction="0.0"/>
   </joint>
   <link
@@ -265,7 +264,6 @@
     <axis
       xyz="0 0 1" />
-    <limit
-      effort="100"
-      velocity="100" />
+    <limit effort="1000000" velocity="10000"/>
+    <dynamics damping="0.0" friction="0.0"/>
   </joint>
   <link
@@ -321,7 +319,6 @@
     <axis
       xyz="0 0 1" />
-    <limit
-      effort="100"
-      velocity="100" />
+    <limit effort="1000000" velocity="10000"/>
+    <dynamics damping="0.0" friction="0.0"/>
   </joint>
   <link
@@ -377,7 +374,6 @@
     <axis
       xyz="0 0 1" />
-    <limit
-      effort="100"
-      velocity="100" />
+    <limit effort="1000000" velocity="10000"/>
+    <dynamics damping="0.0" friction="0.0"/>
   </joint>
   <link

Commit message: UAV px4 control with QGC implemented and tested (PX4-Autopilot and Micro-XRCE-DDS-Agent packages excluded)

File: src/uav_description/urdf/uav.gazebo.xacro (robot description, xacro)
@@ -11,28 +11,28 @@
     <gazebo reference="front_prop_ccw_link">
         <material>${gazebo_black}</material>
-        <mu1>0.1</mu1>
-        <mu2>0.1</mu2>
-        <gravity>true</gravity>
+        <gravity>false</gravity>
+        <self_collide>false</self_collide>
+        <enable_wind>false</enable_wind>
     </gazebo>
     <!-- Front CW -->
     <gazebo reference="front_prop_cw_link">
         <material>${gazebo_black}</material>
-        <mu1>0.1</mu1>
-        <mu2>0.1</mu2>
-        <gravity>true</gravity>
+        <gravity>false</gravity>
+        <self_collide>false</self_collide>
+        <enable_wind>false</enable_wind>
     </gazebo>
     <!-- Back CCW -->
     <gazebo reference="back_prop_ccw_link">
         <material>${gazebo_black}</material>
-        <mu1>0.1</mu1>
-        <mu2>0.1</mu2>
-        <gravity>true</gravity>
+        <gravity>false</gravity>
+        <self_collide>false</self_collide>
+        <enable_wind>false</enable_wind>
     </gazebo>
     <!-- Back CW -->
     <gazebo reference="back_prop_cw_link">
         <material>${gazebo_black}</material>
-        <mu1>0.1</mu1>
-        <mu2>0.1</mu2>
-        <gravity>true</gravity>
+        <gravity>false</gravity>
+        <self_collide>false</self_collide>
+        <enable_wind>false</enable_wind>
     </gazebo>
     <!-- GPS module -->
@@ -78,5 +78,5 @@
             <pose>0 0 0 0 0 0</pose>
             <topic>scan</topic>
-            <update_rate>10</update_rate>
+            <update_rate>50</update_rate>   <!-- 10 -->
             <always_on>true</always_on>
             <visualize>true</visualize>
@@ -120,26 +120,50 @@
     </gazebo>
     <!-- Enables the communication with ros2_control -->
-    <gazebo>
+    <!-- <gazebo>
         <plugin name="gz_ros2_control::GazeboSimROS2ControlPlugin" filename="gz_ros2_control-system">
             <parameters>$(find uav_control)/config/uav_controllers.yaml</parameters>
         </plugin>
-    </gazebo>
+    </gazebo> -->
     <!-- Front CCW motor -->
     <gazebo>
-      <plugin filename="gz-sim-multicopter-motor-model-system" name="gz::sim::systems::MulticopterMotorModel">
+      <plugin filename="gz-sim-multicopter-motor-model-system"
+      name="gz::sim::systems::MulticopterMotorModel">
         <jointName>front_prop_ccw_joint</jointName>
         <linkName>front_prop_ccw_link</linkName>
         <turningDirection>ccw</turningDirection>
         <timeConstantUp>0.0125</timeConstantUp>
+        <timeConstantDown>0.025</timeConstantDown> <!-- 8.54858e-06 -->
+        <maxRotVelocity>1200</maxRotVelocity>
+        <motorConstant>3.0e-05</motorConstant>
+        <momentConstant>0.016</momentConstant>
+        <commandSubTopic>command/motor_speed</commandSubTopic>
+        <!-- <actuator_number>0</actuator_number> -->
+        <motorNumber>0</motorNumber>
+        <rotorDragCoefficient>8.06428e-05</rotorDragCoefficient>
+        <rollingMomentCoefficient>1e-06</rollingMomentCoefficient>
+        <!-- <motorSpeedPubTopic>motor_speed/0</motorSpeedPubTopic> -->
+        <rotorVelocitySlowdownSim>30</rotorVelocitySlowdownSim>
+        <motorType>velocity</motorType>
+      </plugin>
+    </gazebo>
+    <!-- Back CCW motor -->
+    <gazebo>
+      <plugin filename="gz-sim-multicopter-motor-model-system"
+      name="gz::sim::systems::MulticopterMotorModel">
+        <jointName>back_prop_ccw_joint</jointName>
+        <linkName>back_prop_ccw_link</linkName>
+        <turningDirection>ccw</turningDirection>
+        <timeConstantUp>0.0125</timeConstantUp>
         <timeConstantDown>0.025</timeConstantDown>
-        <maxRotVelocity>8000</maxRotVelocity>
-        <motorConstant>3.0e-05</motorConstant>
-        <momentConstant>0.016</momentConstant>
-        <commandSubTopic>gazebo/command/motor_speed</commandSubTopic>
-        <actuator_number>0</actuator_number>
-        <rotorDragCoefficient>8.06428e-05</rotorDragCoefficient>
-        <rollingMomentCoefficient>1e-06</rollingMomentCoefficient>
-        <motorSpeedPubTopic>motor_speed/0</motorSpeedPubTopic>
-        <rotorVelocitySlowdownSim>1</rotorVelocitySlowdownSim>
+        <maxRotVelocity>1200</maxRotVelocity>
+        <motorConstant>3.0e-05</motorConstant>
+        <momentConstant>0.016</momentConstant>
+        <commandSubTopic>command/motor_speed</commandSubTopic>
+        <!-- <actuator_number>2</actuator_number> -->
+        <motorNumber>1</motorNumber>
+        <rotorDragCoefficient>8.06428e-05</rotorDragCoefficient>
+        <rollingMomentCoefficient>1e-06</rollingMomentCoefficient>
+        <!-- <motorSpeedPubTopic>motor_speed/2</motorSpeedPubTopic> -->
+        <rotorVelocitySlowdownSim>30</rotorVelocitySlowdownSim>
         <motorType>velocity</motorType>
       </plugin>
@@ -147,5 +171,6 @@
     <!-- Front CW motor -->
     <gazebo>
-      <plugin filename="gz-sim-multicopter-motor-model-system" name="gz::sim::systems::MulticopterMotorModel">
+      <plugin filename="gz-sim-multicopter-motor-model-system"
+      name="gz::sim::systems::MulticopterMotorModel">
         <jointName>front_prop_cw_joint</jointName>
         <linkName>front_prop_cw_link</linkName>
@@ -153,33 +178,14 @@
         <timeConstantUp>0.0125</timeConstantUp>
         <timeConstantDown>0.025</timeConstantDown>
-        <maxRotVelocity>8000</maxRotVelocity>
-        <motorConstant>3.0e-05</motorConstant>
-        <momentConstant>0.016</momentConstant>
-        <commandSubTopic>gazebo/command/motor_speed</commandSubTopic>
-        <actuator_number>1</actuator_number>
-        <rotorDragCoefficient>8.06428e-05</rotorDragCoefficient>
-        <rollingMomentCoefficient>1e-06</rollingMomentCoefficient>
-        <motorSpeedPubTopic>motor_speed/1</motorSpeedPubTopic>
-        <rotorVelocitySlowdownSim>1</rotorVelocitySlowdownSim>
-        <motorType>velocity</motorType>
-      </plugin>
-    </gazebo>
-    <!-- Back CCW motor -->
-    <gazebo>
-      <plugin filename="gz-sim-multicopter-motor-model-system" name="gz::sim::systems::MulticopterMotorModel">
-        <jointName>back_prop_ccw_joint</jointName>
-        <linkName>back_prop_ccw_link</linkName>
-        <turningDirection>ccw</turningDirection>
-        <timeConstantUp>0.0125</timeConstantUp>
-        <timeConstantDown>0.025</timeConstantDown>
-        <maxRotVelocity>8000</maxRotVelocity>
-        <motorConstant>3.0e-05</motorConstant>
-        <momentConstant>0.016</momentConstant>
-        <commandSubTopic>gazebo/command/motor_speed</commandSubTopic>
-        <actuator_number>2</actuator_number>
-        <rotorDragCoefficient>8.06428e-05</rotorDragCoefficient>
-        <rollingMomentCoefficient>1e-06</rollingMomentCoefficient>
-        <motorSpeedPubTopic>motor_speed/2</motorSpeedPubTopic>
-        <rotorVelocitySlowdownSim>1</rotorVelocitySlowdownSim>
+        <maxRotVelocity>1200</maxRotVelocity>
+        <motorConstant>3.0e-05</motorConstant>
+        <momentConstant>0.016</momentConstant>
+        <commandSubTopic>command/motor_speed</commandSubTopic>
+        <!-- <actuator_number>1</actuator_number> -->
+        <motorNumber>2</motorNumber>
+        <rotorDragCoefficient>8.06428e-05</rotorDragCoefficient>
+        <rollingMomentCoefficient>1e-06</rollingMomentCoefficient>
+        <!-- <motorSpeedPubTopic>motor_speed/1</motorSpeedPubTopic> -->
+        <rotorVelocitySlowdownSim>30</rotorVelocitySlowdownSim>
         <motorType>velocity</motorType>
       </plugin>
@@ -187,5 +193,6 @@
     <!-- Back CW motor -->
     <gazebo>
-      <plugin filename="gz-sim-multicopter-motor-model-system" name="gz::sim::systems::MulticopterMotorModel">
+      <plugin filename="gz-sim-multicopter-motor-model-system"
+      name="gz::sim::systems::MulticopterMotorModel">
         <jointName>back_prop_cw_joint</jointName>
         <linkName>back_prop_cw_link</linkName>
@@ -193,13 +200,14 @@
         <timeConstantUp>0.0125</timeConstantUp>
         <timeConstantDown>0.025</timeConstantDown>
-        <maxRotVelocity>8000</maxRotVelocity>
-        <motorConstant>3.0e-05</motorConstant>
-        <momentConstant>0.016</momentConstant>
-        <commandSubTopic>gazebo/command/motor_speed</commandSubTopic>
-        <actuator_number>3</actuator_number>
-        <rotorDragCoefficient>8.06428e-05</rotorDragCoefficient>
-        <rollingMomentCoefficient>1e-06</rollingMomentCoefficient>
-        <motorSpeedPubTopic>motor_speed/3</motorSpeedPubTopic>
-        <rotorVelocitySlowdownSim>1</rotorVelocitySlowdownSim>
+        <maxRotVelocity>1200</maxRotVelocity>
+        <motorConstant>3.0e-05</motorConstant>
+        <momentConstant>0.016</momentConstant>
+        <commandSubTopic>command/motor_speed</commandSubTopic>
+        <!-- <actuator_number>3</actuator_number> -->
+        <motorNumber>3</motorNumber>
+        <rotorDragCoefficient>8.06428e-05</rotorDragCoefficient>
+        <rollingMomentCoefficient>1e-06</rollingMomentCoefficient>
+        <!-- <motorSpeedPubTopic>motor_speed/3</motorSpeedPubTopic> -->
+        <rotorVelocitySlowdownSim>30</rotorVelocitySlowdownSim>
         <motorType>velocity</motorType>
       </plugin>

File: src/uav_description/urdf/uav.urdf.xacro (robot description, xacro)
@@ -6,6 +6,6 @@
   <xacro:include filename="$(find uav_description)/urdf/core.xacro"/>
   <xacro:include filename="$(find uav_description)/urdf/uav.gazebo.xacro"/>
-  <xacro:include filename="$(find uav_description)/urdf/uav.ros2_control.xacro"/>
-  <link name="base_footprint"/>
+  <!-- <xacro:include filename="$(find uav_description)/urdf/uav.ros2_control.xacro"/> -->
+  <!-- <link name="base_footprint"/> -->
   <link name="base_link">
     <inertial>
@@ -45,10 +45,10 @@
     </collision>
   </link>
-  <joint name="base_footprint_joint"
+  <!-- <joint name="base_footprint_joint"
     type="fixed">
     <origin xyz="0 0 0" rpy="0 0 0" />
     <parent link="base_footprint" />
     <child link="base_link" />
-  </joint>
+  </joint> -->
   <link
     name="lidar_link">
@@ -202,5 +202,5 @@
     <origin
       xyz="0.22481 -0.23326 0.086028"
-      rpy="-0.061392 0.0028205 -2.7734" />
+      rpy="0 0 0" />
     <parent
       link="base_link" />
@@ -209,5 +209,60 @@
     <axis
       xyz="0 0 1" />
-    <limit effort="1000000" velocity="10000"/>
+    <limit effort="1e12" velocity="1e12"/>
+    <dynamics damping="0.0" friction="0.0"/>
+  </joint>
+  <link
+    name="front_prop_cw_link">
+    <inertial>
+      <origin
+        xyz="1.89889458346304E-06 -0.000131188965704798 0.00588670324654172"
+        rpy="0 0 0" />
+      <mass
+        value="0.0232860557198823" />
+      <inertia
+        ixx="6.48761674575812E-07"
+        ixy="-1.71419194967408E-07"
+        ixz="1.28654962833368E-10"
+        iyy="2.84759689374051E-05"
+        iyz="5.39216374404741E-11"
+        izz="2.90785252715597E-05" />
+    </inertial>
+    <visual>
+      <origin
+        xyz="0 0 0"
+        rpy="0 0 0" />
+      <geometry>
+        <mesh
+          filename="file://$(find uav_description)/meshes/front_prop_cw_link.STL" />
+      </geometry>
+      <material
+        name="">
+        <color
+          rgba="0.752941176470588 0.752941176470588 0.752941176470588 1" />
+      </material>
+    </visual>
+    <collision>
+      <origin
+        xyz="0 0 0"
+        rpy="0 0 0" />
+      <geometry>
+        <mesh
+          filename="file://$(find uav_description)/meshes/front_prop_cw_link.STL" />
+      </geometry>
+    </collision>
+  </link>
+  <joint
+    name="front_prop_cw_joint"
+    type="continuous">
+    <origin
+      xyz="0.23106 0.22649 0.090005"
+      rpy="0 0 0" />
+    <parent
+      link="base_link" />
+    <child
+      link="front_prop_cw_link" />
+    <axis
+      xyz="0 0 1" />
+    <limit effort="1e12" velocity="1e12"/>
     <dynamics damping="0.0" friction="0.0"/>
   </joint>
@@ -257,5 +312,5 @@
     <origin
       xyz="-0.2287 0.23276 0.086501"
-      rpy="-0.062752 0.0019097 -3.0845" />
+      rpy="0 0 0" />
     <parent
       link="base_link" />
@@ -264,60 +319,5 @@
     <axis
       xyz="0 0 1" />
-    <limit effort="1000000" velocity="10000"/>
-    <dynamics damping="0.0" friction="0.0"/>
-  </joint>
-  <link
-    name="front_prop_cw_link">
-    <inertial>
-      <origin
-        xyz="1.89889458346304E-06 -0.000131188965704798 0.00588670324654172"
-        rpy="0 0 0" />
-      <mass
-        value="0.0232860557198823" />
-      <inertia
-        ixx="6.48761674575812E-07"
-        ixy="-1.71419194967408E-07"
-        ixz="1.28654962833368E-10"
-        iyy="2.84759689374051E-05"
-        iyz="5.39216374404741E-11"
-        izz="2.90785252715597E-05" />
-    </inertial>
-    <visual>
-      <origin
-        xyz="0 0 0"
-        rpy="0 0 0" />
-      <geometry>
-        <mesh
-          filename="file://$(find uav_description)/meshes/front_prop_cw_link.STL" />
-      </geometry>
-      <material
-        name="">
-        <color
-          rgba="0.752941176470588 0.752941176470588 0.752941176470588 1" />
-      </material>
-    </visual>
-    <collision>
-      <origin
-        xyz="0 0 0"
-        rpy="0 0 0" />
-      <geometry>
-        <mesh
-          filename="file://$(find uav_description)/meshes/front_prop_cw_link.STL" />
-      </geometry>
-    </collision>
-  </link>
-  <joint
-    name="front_prop_cw_joint"
-    type="continuous">
-    <origin
-      xyz="0.23106 0.22649 0.090005"
-      rpy="-0.0032394 0.0041761 -2.9988" />
-    <parent
-      link="base_link" />
-    <child
-      link="front_prop_cw_link" />
-    <axis
-      xyz="0 0 1" />
-    <limit effort="1000000" velocity="10000"/>
+    <limit effort="1e12" velocity="1e12"/>
     <dynamics damping="0.0" friction="0.0"/>
   </joint>
@@ -367,5 +367,5 @@
     <origin
       xyz="-0.23496 -0.22701 0.086701"
-      rpy="-0.003654 0.0038186 -3.1024" />
+      rpy="0 0 0" />
     <parent
       link="base_link" />
@@ -374,5 +374,5 @@
     <axis
       xyz="0 0 1" />
-    <limit effort="1000000" velocity="10000"/>
+    <limit effort="1e12" velocity="1e12"/>
     <dynamics damping="0.0" friction="0.0"/>
   </joint>
