Commit message: Multiple tf trees problem fixed, xacro for future multicopter usage prepared.

File: src/uav_description/urdf/uav.gazebo.xacro (robot description, xacro)
@@ -2,5 +2,5 @@
 <robot name="uav" xmlns:xacro="http://ros.org/wiki/xacro">
     <!-- Base link -->
-    <gazebo reference="base_link">
+    <gazebo reference="x650_0/base_link">
         <material>${gazebo_grey}</material>
         <mu1>0.1</mu1>
@@ -9,5 +9,5 @@
     </gazebo>
     <!-- Front CCW -->
-    <gazebo reference="front_prop_ccw_link">
+    <gazebo reference="x650_0/front_prop_ccw_link">
         <material>${gazebo_black}</material>
         <gravity>false</gravity>
@@ -16,5 +16,5 @@
     </gazebo>
     <!-- Front CW -->
-    <gazebo reference="front_prop_cw_link">
+    <gazebo reference="x650_0/front_prop_cw_link">
         <material>${gazebo_black}</material>
         <gravity>false</gravity>
@@ -23,5 +23,5 @@
     </gazebo>
     <!-- Back CCW -->
-    <gazebo reference="back_prop_ccw_link">
+    <gazebo reference="x650_0/back_prop_ccw_link">
         <material>${gazebo_black}</material>
         <gravity>false</gravity>
@@ -30,5 +30,5 @@
     </gazebo>
     <!-- Back CW -->
-    <gazebo reference="back_prop_cw_link">
+    <gazebo reference="x650_0/back_prop_cw_link">
         <material>${gazebo_black}</material>
         <gravity>false</gravity>
@@ -37,5 +37,5 @@
     </gazebo>
     <!-- GPS module -->
-    <gazebo reference="gps_module_link">
+    <gazebo reference="x650_0/gps_module_link">
         <material>${gazebo_black}</material>
         <mu1>0.1</mu1>
@@ -44,5 +44,5 @@
     </gazebo>
     <!-- Depth camera -->
-    <gazebo reference="depth_camera_link">
+    <gazebo reference="x650_0/depth_camera_link">
         <material>${gazebo_white}</material>
         <mu1>0.1</mu1>
@@ -70,5 +70,5 @@
     </gazebo>
     <!-- Lidar sensor -->
-    <gazebo reference="lidar_link">
+    <gazebo reference="x650_0/lidar_link">
         <material>${gazebo_dark_grey}</material>
         <mu1>0.1</mu1>
@@ -129,6 +129,6 @@
       <plugin filename="gz-sim-multicopter-motor-model-system"
       name="gz::sim::systems::MulticopterMotorModel">
-        <jointName>front_prop_ccw_joint</jointName>
-        <linkName>front_prop_ccw_link</linkName>
+        <jointName>x650_0/front_prop_ccw_joint</jointName>
+        <linkName>x650_0/front_prop_ccw_link</linkName>
         <turningDirection>ccw</turningDirection>
         <timeConstantUp>0.0125</timeConstantUp>
@@ -151,6 +151,6 @@
       <plugin filename="gz-sim-multicopter-motor-model-system"
       name="gz::sim::systems::MulticopterMotorModel">
-        <jointName>back_prop_ccw_joint</jointName>
-        <linkName>back_prop_ccw_link</linkName>
+        <jointName>x650_0/back_prop_ccw_joint</jointName>
+        <linkName>x650_0/back_prop_ccw_link</linkName>
         <turningDirection>ccw</turningDirection>
         <timeConstantUp>0.0125</timeConstantUp>
@@ -173,6 +173,6 @@
       <plugin filename="gz-sim-multicopter-motor-model-system"
       name="gz::sim::systems::MulticopterMotorModel">
-        <jointName>front_prop_cw_joint</jointName>
-        <linkName>front_prop_cw_link</linkName>
+        <jointName>x650_0/front_prop_cw_joint</jointName>
+        <linkName>x650_0/front_prop_cw_link</linkName>
         <turningDirection>cw</turningDirection>
         <timeConstantUp>0.0125</timeConstantUp>
@@ -195,6 +195,6 @@
       <plugin filename="gz-sim-multicopter-motor-model-system"
       name="gz::sim::systems::MulticopterMotorModel">
-        <jointName>back_prop_cw_joint</jointName>
-        <linkName>back_prop_cw_link</linkName>
+        <jointName>x650_0/back_prop_cw_joint</jointName>
+        <linkName>x650_0/back_prop_cw_link</linkName>
         <turningDirection>cw</turningDirection>
         <timeConstantUp>0.0125</timeConstantUp>

File: src/uav_description/urdf/uav.urdf.xacro (robot description, xacro)
@@ -7,11 +7,11 @@
   <xacro:include filename="$(find uav_description)/urdf/uav.gazebo.xacro"/>
   <!-- <xacro:include filename="$(find uav_description)/urdf/uav.ros2_control.xacro"/> -->
-  <link name="base_footprint"/>
-  <joint name="base_footprint_joint" type="fixed">
+  <link name="x650_0/base_footprint"/>
+  <joint name="x650_0/base_footprint_joint" type="fixed">
     <origin xyz="0 0 0" rpy="0 0 0" />
-    <parent link="base_footprint" />
-    <child link="base_link" />
-  </joint>
-  <link name="base_link">
+    <parent link="x650_0/base_footprint" />
+    <child link="x650_0/base_link" />
+  </joint>
+  <link name="x650_0/base_link">
     <inertial>
       <origin
@@ -51,5 +51,5 @@
   </link>
   <link
-    name="lidar_link">
+    name="x650_0/lidar_link">
     <inertial>
       <origin
@@ -91,5 +91,5 @@
   </link>
   <joint
-    name="lidar_joint"
+    name="x650_0/lidar_joint"
     type="fixed">
     <origin
@@ -97,12 +97,12 @@
       rpy="0.0038504 -0.0036204 -0.013619" />
     <parent
-      link="base_link" />
-    <child
-      link="lidar_link" />
+      link="x650_0/base_link" />
+    <child
+      link="x650_0/lidar_link" />
     <axis
       xyz="0 0 0" />
   </joint>
   <!-- LiDAR link -->
-  <link name="laser_sensor_link">
+  <link name="x650_0/laser_sensor_link">
     <visual>
       <geometry>
@@ -111,11 +111,11 @@
     </visual>
   </link>
-  <joint name="laser_sensor_joint" type="fixed">
-    <parent link="base_link"/>
-    <child link="laser_sensor_link"/>
+  <joint name="x650_0/laser_sensor_joint" type="fixed">
+    <parent link="x650_0/base_link"/>
+    <child link="x650_0/laser_sensor_link"/>
     <origin xyz="0 0 0.15" rpy="0 0 0"/>
   </joint>
   <link
-    name="gps_module_link">
+    name="x650_0/gps_module_link">
     <inertial>
       <origin
@@ -157,5 +157,5 @@
   </link>
   <joint
-    name="gps_module_joint"
+    name="x650_0/gps_module_joint"
     type="fixed">
     <origin
@@ -163,12 +163,12 @@
       rpy="0.0025723 0.004617 -1.8307" />
     <parent
-      link="base_link" />
-    <child
-      link="gps_module_link" />
+      link="x650_0/base_link" />
+    <child
+      link="x650_0/gps_module_link" />
     <axis
       xyz="0 0 0" />
   </joint>
   <link
-    name="front_prop_ccw_link">
+    name="x650_0/front_prop_ccw_link">
     <inertial>
       <origin
@@ -210,5 +210,5 @@
   </link>
   <joint
-    name="front_prop_ccw_joint"
+    name="x650_0/front_prop_ccw_joint"
     type="continuous">
     <origin
@@ -216,7 +216,7 @@
       rpy="0 0 0" />
     <parent
-      link="base_link" />
-    <child
-      link="front_prop_ccw_link" />
+      link="x650_0/base_link" />
+    <child
+      link="x650_0/front_prop_ccw_link" />
     <axis
       xyz="0 0 1" />
@@ -225,5 +225,5 @@
   </joint>
   <link
-    name="front_prop_cw_link">
+    name="x650_0/front_prop_cw_link">
     <inertial>
       <origin
@@ -265,5 +265,5 @@
   </link>
   <joint
-    name="front_prop_cw_joint"
+    name="x650_0/front_prop_cw_joint"
     type="continuous">
     <origin
@@ -271,7 +271,7 @@
       rpy="0 0 0" />
     <parent
-      link="base_link" />
-    <child
-      link="front_prop_cw_link" />
+      link="x650_0/base_link" />
+    <child
+      link="x650_0/front_prop_cw_link" />
     <axis
       xyz="0 0 1" />
@@ -280,5 +280,5 @@
   </joint>
   <link
-    name="back_prop_ccw_link">
+    name="x650_0/back_prop_ccw_link">
     <inertial>
       <origin
@@ -320,5 +320,5 @@
   </link>
   <joint
-    name="back_prop_ccw_joint"
+    name="x650_0/back_prop_ccw_joint"
     type="continuous">
     <origin
@@ -326,7 +326,7 @@
       rpy="0 0 0" />
     <parent
-      link="base_link" />
-    <child
-      link="back_prop_ccw_link" />
+      link="x650_0/base_link" />
+    <child
+      link="x650_0/back_prop_ccw_link" />
     <axis
       xyz="0 0 1" />
@@ -335,5 +335,5 @@
   </joint>
   <link
-    name="back_prop_cw_link">
+    name="x650_0/back_prop_cw_link">
     <inertial>
       <origin
@@ -375,5 +375,5 @@
   </link>
   <joint
-    name="back_prop_cw_joint"
+    name="x650_0/back_prop_cw_joint"
     type="continuous">
     <origin
@@ -381,7 +381,7 @@
       rpy="0 0 0" />
     <parent
-      link="base_link" />
-    <child
-      link="back_prop_cw_link" />
+      link="x650_0/base_link" />
+    <child
+      link="x650_0/back_prop_cw_link" />
     <axis
       xyz="0 0 1" />
@@ -390,5 +390,5 @@
   </joint>
   <link
-    name="depth_camera_link">
+    name="x650_0/depth_camera_link">
     <inertial>
       <origin
@@ -430,5 +430,5 @@
   </link>
   <joint
-    name="depth_camera_joint"
+    name="x650_0/depth_camera_joint"
     type="fixed">
     <origin
@@ -436,7 +436,7 @@
       rpy="-3.1377 -0.0036204 -0.013619" />
     <parent
-      link="base_link" />
-    <child
-      link="depth_camera_link" />
+      link="x650_0/base_link" />
+    <child
+      link="x650_0/depth_camera_link" />
     <axis
       xyz="0 0 0" />

Commit message: GPS issue in gazebo fixed

File: src/uav_description/urdf/uav.gazebo.xacro (robot description, xacro)
@@ -1,16 +1,4 @@
 <?xml version="1.0"?>
 <robot name="uav_uav" xmlns:xacro="http://ros.org/wiki/xacro">
-    <gazebo reference="back_prop_cw_link">
-        <material>${gazebo_black}</material>
-        <mu1>0.1</mu1>
-        <mu2>0.1</mu2>
-        <gravity>true</gravity>
-    </gazebo>
-    <gazebo reference="back_prop_ccw_link">
-        <material>${gazebo_black}</material>
-        <mu1>0.1</mu1>
-        <mu2>0.1</mu2>
-        <gravity>true</gravity>
-    </gazebo>
     <!-- Base link -->
     <gazebo reference="base_link">
@@ -98,11 +86,4 @@
     <!-- Telemetry -->
     <gazebo reference="telemetry_link">
-        <material>${gazebo_black}</material>
-        <mu1>0.1</mu1>
-        <mu2>0.1</mu2>
-        <gravity>true</gravity>
-    </gazebo>
-    <!-- GPS module -->
-    <gazebo reference="gps_module_link">
         <material>${gazebo_black}</material>
         <mu1>0.1</mu1>
@@ -131,4 +112,33 @@
         <gravity>true</gravity>
     </gazebo>
+    <!-- GPS module -->
+    <gazebo reference="gps_module_link">
+        <material>${gazebo_black}</material>
+        <mu1>0.1</mu1>
+        <mu2>0.1</mu2>
+        <gravity>true</gravity>
+        <sensor name="navsat" type="navsat">
+            <always_on>true</always_on>
+            <update_rate>1</update_rate>
+            <topic>/gps/fix</topic>
+            <gz_frame_id>gps_module_link</gz_frame_id>
+            <navsat>
+                <position_sensing>
+                <horizontal>
+                    <noise type="gaussian">
+                    <mean>0.0</mean>
+                    <stddev>0.0</stddev>
+                    </noise>
+                </horizontal>
+                <vertical>
+                    <noise type="gaussian">
+                    <mean>0.0</mean>
+                    <stddev>0.0</stddev>
+                    </noise>
+                </vertical>
+                </position_sensing>
+            </navsat>
+        </sensor>
+    </gazebo>
     <!-- Depth camera -->
     <gazebo reference="depth_camera_link">
@@ -138,6 +148,7 @@
         <gravity>true</gravity>
         <sensor name="rgbd_cam" type="rgbd_camera">
+            <pose>0 0 0 0 0 0</pose>
             <camera>
-                <horizontal_fov>1.5184</horizontal_fov>
+                <horizontal_fov>1.2</horizontal_fov>
                 <image>
                     <width>600</width>
@@ -147,11 +158,12 @@
                 <clip>
                     <near>0.6</near>
-                    <far>6.0</far>
+                    <far>100.0</far>    <!-- Note: This is set to 100, otherwise the scene gets clipped -->
                 </clip>
+                <point_cloud>true</point_cloud>
             </camera>
-            <always_on>1</always_on>
+            <always_on>true</always_on>
             <gz_frame_id>depth_camera_link</gz_frame_id>
             <topic>camera</topic>
-            <update_rate>15.0</update_rate>
+            <update_rate>5</update_rate>
             <visualize>true</visualize>
         </sensor>
@@ -164,7 +176,7 @@
         <gravity>true</gravity>
         <sensor name="laser_sensor" type="gpu_lidar">
-            <pose>0 0 0 0 0 0</pose>
+            <pose>-0.00044268 -0.00016922 0.12747 0.0038504 -0.0036204 -0.013619</pose>
             <topic>scan</topic>
-            <update_rate>10</update_rate>
+            <update_rate>5</update_rate>
             <always_on>true</always_on>
             <visualize>true</visualize>
@@ -173,24 +185,78 @@
                 <scan>
                     <horizontal>
-                        <!-- Based on technical specs -->
-                        <samples>720</samples>
+                        <samples>360</samples>
                         <resolution>1</resolution>
-                        <min_angle>-3.14159</min_angle>
-                        <max_angle>3.14159</max_angle>
+                        <min_angle>0.000000</min_angle>
+                        <max_angle>6.280000</max_angle>
                     </horizontal>
-                    <!-- 2D Lidar settings -->
                     <vertical>
                         <samples>1</samples>
                         <resolution>1</resolution>
-                        <min_angle>0.0</min_angle>
-                        <max_angle>0.0</max_angle>
+                        <min_angle>0</min_angle>
+                        <max_angle>0</max_angle>
                     </vertical>
                 </scan>
                 <range>
-                    <min>0.15</min>
-                    <max>6.0</max>
+                    <min>0.2</min>
+                    <max>12.0</max>
                     <resolution>0.001</resolution>
                 </range>
+                <noise>
+                    <type>gaussian</type>
+                    <mean>0.0</mean>
+                    <stddev>0.01</stddev>
+                </noise>
             </lidar>
+        </sensor>
+    </gazebo>
+    <!-- IMU sensor -->
+    <gazebo reference="pixhawk_jetson_mc_link">
+        <sensor name="imu_sensor" type="imu">
+            <always_on>true</always_on>
+            <update_rate>100</update_rate>
+            <topic>/imu/data</topic>
+            <gz_frame_id>pixhawk_jetson_mc_link</gz_frame_id>
+            <imu>
+            <angular_velocity>
+                <x>
+                <noise type="gaussian">
+                    <mean>0.0</mean>
+                    <stddev>2e-4</stddev>
+                </noise>
+                </x>
+                <y>
+                <noise type="gaussian">
+                    <mean>0.0</mean>
+                    <stddev>2e-4</stddev>
+                </noise>
+                </y>
+                <z>
+                <noise type="gaussian">
+                    <mean>0.0</mean>
+                    <stddev>2e-4</stddev>
+                </noise>
+                </z>
+            </angular_velocity>
+            <linear_acceleration>
+                <x>
+                <noise type="gaussian">
+                    <mean>0.0</mean>
+                    <stddev>1.7e-2</stddev>
+                </noise>
+                </x>
+                <y>
+                <noise type="gaussian">
+                    <mean>0.0</mean>
+                    <stddev>1.7e-2</stddev>
+                </noise>
+                </y>
+                <z>
+                <noise type="gaussian">
+                    <mean>0.0</mean>
+                    <stddev>1.7e-2</stddev>
+                </noise>
+                </z>
+            </linear_acceleration>
+            </imu>
         </sensor>
     </gazebo>
